File: KiCad/GN10Mainboard/GN10Mainboard.kicad_sch (KiCad schematic)
At the start: 132 parts, among them J1 XT30PW-M, J2 Conn_01x02_Pin, J3 USB_C_Receptacle_USB2.0_16P, J4 Conn_01x04, J5 Conn_01x04, J6 Conn_01x04, J7 Conn_01x04, J8 Conn_01x04, J9 Conn_01x06, SW1 SW_Push, SW2 SW_DIP_x04, SW3 SW_Push, SW4 SW_Push, U1 OKL-T/x-W5N-C, U10 BNO055, U2 3.3V, U3 STM32G474RCTx, U4 TBD62083AFNG, U5 7segmentLED, U6 RNBD451, U7 FT2232HQ, U8 MCP2562-E-SN, U9 MCP2562-E-SN, Y1 24MHz, Y2 Crystal, Y3 32.768kHz, Y4 12M

Commit message: PCB: I wired 70% of parts but placement is bad. So I'll redo.
Connections:
- net CAN2_RX: now also U8.1 (TXD); no longer U9.1 (TXD)
- net CAN2_TX: now also U8.4 (RXD); no longer U9.4 (RXD)
- net CAN3_RX: now also U9.1 (TXD); no longer U8.1 (TXD)
- net CAN3_TX: now also U9.4 (RXD); no longer U8.4 (RXD)
- net CAN3_H renamed CAN1_H
- net CAN3_L renamed CAN1_L
Changed lines of the file:
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@@
+		)
+	)
+	(global_label "CAN3_RX"
+		(shape output)
+		(at 483.87 287.02 180)
+		(fields_autoplaced yes)
+		(effects
+			(font
+				(size 1.27 1.27)
+			)
+			(justify right)
+		)
+		(property "Intersheetrefs" "${INTERSHEET_REFS}"
+			(at 472.5391 287.02 0)
+			(effects
+				(font
+					(size 1.27 1.27)
+				)
+				(justify right)
+				(hide yes)
+			)
 		)
 	)
@@
 		)
 	)
-	(global_label "CAN3_H"
+	(global_label "CAN1_H"
 		(shape passive)
 		(at 509.27 220.98 0)
@@
 		(property "Intersheetrefs" "${INTERSHEET_REFS}"
 			(at 199.6101 201.93 0)
-			(effects
-				(font
-					(size 1.27 1.27)
-				)
-				(justify right)
-				(hide yes)
-			)
-		)
-	)
-	(global_label "CAN3_RX"
-		(shape output)
-		(at 483.87 218.44 180)
-		(fields_autoplaced yes)
-		(effects
-			(font
-				(size 1.27 1.27)
-			)
-			(justify right)
-		)
-		(property "Intersheetrefs" "${INTERSHEET_REFS}"
-			(at 472.5391 218.44 0)
 			(effects
 				(font
@@
 		)
 	)
+	(global_label "CAN3_TX"
+		(shape input)
+		(at 483.87 289.56 180)
+		(fields_autoplaced yes)
+		(effects
+			(font
+				(size 1.27 1.27)
+			)
+			(justify right)
+		)
+		(property "Intersheetrefs" "${INTERSHEET_REFS}"
+			(at 472.8415 289.56 0)
+			(effects
+				(font
+					(size 1.27 1.27)
+				)
+				(justify right)
+				(hide yes)
+			)
+		)
+	)
 	(global_label "SPI3_MISO"
 		(shape output)
@@
 		)
 	)
-	(global_label "CAN3_L"
+	(global_label "CAN1_L"
 		(shape passive)
 		(at 509.27 226.06 0)
@@
 		)
 	)
-	(global_label "CAN2_RX"
-		(shape output)
-		(at 483.87 287.02 180)
-		(fields_autoplaced yes)
-		(effects
-			(font
-				(size 1.27 1.27)
-			)
-			(justify right)
-		)
-		(property "Intersheetrefs" "${INTERSHEET_REFS}"
-			(at 472.5391 287.02 0)
-			(effects
-				(font
-					(size 1.27 1.27)
-				)
-				(justify right)
-				(hide yes)
-			)
-		)
-	)
-	(global_label "CAN3_TX"
-		(shape input)
-		(at 483.87 220.98 180)
-		(fields_autoplaced yes)
-		(effects
-			(font
-				(size 1.27 1.27)
-			)
-			(justify right)
-		)
-		(property "Intersheetrefs" "${INTERSHEET_REFS}"
-			(at 472.8415 220.98 0)
-			(effects
-				(font
-					(size 1.27 1.27)
-				)
-				(justify right)
-				(hide yes)
-			)
-		)
-	)
 	(global_label "BLE_DEBUG_UART_RX"
 		(shape output)
@@
 		)
 	)
-	(global_label "CAN3_L"
+	(global_label "CAN1_L"
 		(shape passive)
 		(at 543.56 222.25 0)
@@
 		)
 	)
+	(global_label "USART1_CTS"
+		(shape input)
+		(at 109.22 227.33 0)
+		(fields_autoplaced yes)
+		(effects
+			(font
+				(size 1.27 1.27)
+			)
+			(justify left)
+		)
+		(property "Intersheetrefs" "${INTERSHEET_REFS}"
+			(at 123.6956 227.33 0)
+			(effects
+				(font
+					(size 1.27 1.27)
+				)
+				(justify left)
+				(hide yes)
+			)
+		)
+	)
+	(global_label "USART3_TX"
+		(shape input)
+		(at 54.61 372.11 180)
+		(fields_autoplaced yes)
+		(effects
+			(font
+				(size 1.27 1.27)
+			)
+			(justify right)
+		)
+		(property "Intersheetrefs" "${INTERSHEET_REFS}"
+			(at 41.4044 372.11 0)
+			(effects
+				(font
+					(size 1.27 1.27)
+				)
+				(justify right)
+				(hide yes)
+			)
+		)
+	)
+	(global_label "BLE_UART_CTS"
+		(shape output)
+		(at 347.98 358.14 0)
+		(fields_autoplaced yes)
+		(effects
+			(font
+				(size 1.27 1.27)
+			)
+			(justify left)
+		)
+		(property "Intersheetrefs" "${INTERSHEET_REFS}"
+			(at 364.4513 358.14 0)
+			(effects
+				(font
+					(size 1.27 1.27)
+				)
+				(justify left)
+				(hide yes)
+			)
+		)
+	)
+	(global_label "LED_F_DRV"
+		(shape input)
+		(at 207.01 232.41 180)
+		(fields_autoplaced yes)
+		(effects
+			(font
+				(size 1.27 1.27)
+			)
+			(justify right)
+		)
+		(property "Intersheetrefs" "${INTERSHEET_REFS}"
+			(at 193.9253 232.41 0)
+			(effects
+				(font
+					(size 1.27 1.27)
+				)
+				(justify right)
+				(hide yes)
+			)
+		)
+	)
 	(global_label "CAN2_TX"
 		(shape input)
-		(at 483.87 289.56 180)
-		(fields_autoplaced yes)
-		(effects
-			(font
-				(size 1.27 1.27)
-			)
-			(justify right)
-		)
-		(property "Intersheetrefs" "${INTERSHEET_REFS}"
-			(at 472.8415 289.56 0)
-			(effects
-				(font
-					(size 1.27 1.27)
-				)
-				(justify right)
-				(hide yes)
-			)
-		)
-	)
-	(global_label "USART1_CTS"
-		(shape input)
-		(at 109.22 227.33 0)
-		(fields_autoplaced yes)
-		(effects
-			(font
-				(size 1.27 1.27)
-			)
-			(justify left)
-		)
-		(property "Intersheetrefs" "${INTERSHEET_REFS}"
-			(at 123.6956 227.33 0)
-			(effects
-				(font
-					(size 1.27 1.27)
-				)
-				(justify left)
-				(hide yes)
-			)
-		)
-	)
-	(global_label "USART3_TX"
-		(shape input)
-		(at 54.61 372.11 180)
-		(fields_autoplaced yes)
-		(effects
-			(font
-				(size 1.27 1.27)
-			)
-			(justify right)
-		)
-		(property "Intersheetrefs" "${INTERSHEET_REFS}"
-			(at 41.4044 372.11 0)
-			(effects
-				(font
-					(size 1.27 1.27)
-				)
-				(justify right)
-				(hide yes)
-			)
-		)
-	)
-	(global_label "BLE_UART_CTS"
-		(shape output)
-		(at 347.98 358.14 0)
-		(fields_autoplaced yes)
-		(effects
-			(font
-				(size 1.27 1.27)
-			)
-			(justify left)
-		)
-		(property "Intersheetrefs" "${INTERSHEET_REFS}"
-			(at 364.4513 358.14 0)
-			(effects
-				(font
-					(size 1.27 1.27)
-				)
-				(justify left)
-				(hide yes)
-			)
-		)
-	)
-	(global_label "LED_F_DRV"
-		(shape input)
-		(at 207.01 232.41 180)
-		(fields_autoplaced yes)
-		(effects
-			(font
-				(size 1.27 1.27)
-			)
-			(justify right)
-		)
-		(property "Intersheetrefs" "${INTERSHEET_REFS}"
-			(at 193.9253 232.41 0)
+		(at 483.87 220.98 180)
+		(fields_autoplaced yes)
+		(effects
+			(font
+				(size 1.27 1.27)
+			)
+			(justify right)
+		)
+		(property "Intersheetrefs" "${INTERSHEET_REFS}"
+			(at 472.8415 220.98 0)
 			(effects
 				(font
@@
 		)
 	)
+	(global_label "CAN2_RX"
+		(shape output)
+		(at 483.87 218.44 180)
+		(fields_autoplaced yes)
+		(effects
+			(font
+				(size 1.27 1.27)
+			)
+			(justify right)
+		)
+		(property "Intersheetrefs" "${INTERSHEET_REFS}"
+			(at 472.5391 218.44 0)
+			(effects
+				(font
+					(size 1.27 1.27)
+				)
+				(justify right)
+				(hide yes)
+			)
+		)
+	)
 	(global_label "DIP_4"
 		(shape input)
@@
 		)
 	)
-	(global_label "CAN3_H"
+	(global_label "CAN1_H"
 		(shape passive)
 		(at 543.56 217.17 0)

Commit message: Wiring complete
Parts:
- removed D17: White, LED_SMD:LED_0603_1608Metric_Pad1.05x0.95mm_HandSolder, symbol Device:LED
- removed D6: Red, LED_SMD:LED_0603_1608Metric_Pad1.05x0.95mm_HandSolder, symbol Device:LED
- removed R33, R9: 1k, Resistor_SMD:R_0603_1608Metric_Pad0.98x0.95mm_HandSolder, symbol Device:R
Connections:
- net DIP_4: now also U3.17 (PA3); no longer U3.14 (PA2)
- no-connect marks 55 -> 56

Commit message: update ioc and clean chematic for v1.0
Parts:
- removed C21, C23, C26, C27, C29, C31, C32, C33, C34: 0.1u, Capacitor_SMD:C_0402_1005Metric_Pad0.74x0.62mm_HandSolder, symbol Device:C
- removed C22: 4.7u, Resistor_SMD:R_0603_1608Metric_Pad0.98x0.95mm_HandSolder, symbol Device:C
- removed C24, C25: 10u, Capacitor_SMD:C_0603_1608Metric_Pad1.08x0.95mm_HandSolder, symbol Device:C
- removed C28, C30: 1u, Capacitor_SMD:C_0402_1005Metric_Pad0.74x0.62mm_HandSolder, symbol Device:C
- removed D13, D14: Green, LED_SMD:LED_0603_1608Metric_Pad1.05x0.95mm_HandSolder, symbol Device:LED
- removed D15, D16: Blue, LED_SMD:LED_0603_1608Metric_Pad1.05x0.95mm_HandSolder, symbol Device:LED
- removed D5: White, LED_SMD:LED_0603_1608Metric_Pad1.05x0.95mm_HandSolder, symbol Device:LED
- removed J3: USB_C_Receptacle_USB2.0_16P, Connector_USB:USB_C_Receptacle_HRO_TYPE-C-31-M-12, symbol Connector:USB_C_Receptacle_USB2.0_16P
- removed JP10, JP2, JP7, JP8, JP9: SolderJumper_2_Open, Jumper:SolderJumper-2_P1.3mm_Open_RoundedPad1.0x1.5mm, symbol Jumper:SolderJumper_2_Open
- removed L1, L2: 0.47u, Inductor_SMD:L_0603_1608Metric_Pad1.05x0.95mm_HandSolder, symbol Device:L
- removed R20: 10k, Resistor_SMD:R_0603_1608Metric_Pad0.98x0.95mm_HandSolder, symbol Device:R
- removed R25, R26: 4.7k, Resistor_SMD:R_0402_1005Metric_Pad0.72x0.64mm_HandSolder, symbol Device:R
- removed R27: 1k, Resistor_SMD:R_0402_1005Metric_Pad0.72x0.64mm_HandSolder, symbol Device:R
- removed R28: 12k, Resistor_SMD:R_0402_1005Metric_Pad0.72x0.64mm_HandSolder, symbol Device:R
- removed R29, R30, R31, R32: 470, Resistor_SMD:R_0603_1608Metric_Pad0.98x0.95mm_HandSolder, symbol Device:R
- removed R7: 1k, Resistor_SMD:R_0603_1608Metric_Pad0.98x0.95mm_HandSolder, symbol Device:R
- removed SW4: SW_Push, GN10_Parts:TVAF, symbol Switch:SW_Push
- removed U10: BNO055, GN10_Parts:BNO055, symbol GN10_Parts:BNO055
- removed U7: FT2232HQ, Package_DFN_QFN:QFN-64-1EP_9x9mm_P0.5mm_EP4.35x4.35mm, symbol Interface_USB:FT2232HQ
- removed Y4: 12M, Crystal:Resonator_SMD_Murata_CSTxExxV-3Pin_3.0x1.1mm_HandSoldering, symbol Device:Crystal_GND2
- added D6: Green, LED_SMD:LED_0603_1608Metric_Pad1.05x0.95mm_HandSolder, symbol Device:LED
- added R9: 1k, Resistor_SMD:R_0603_1608Metric_Pad0.98x0.95mm_HandSolder, symbol Device:R
Connections:
- net GND: now also R9.2
- net LED_RED: now also D6.2 (A)
- new net: D6.1 (K), R9.1
- no-connect marks 56 -> 26
Other:
- note removed: "Gyro Sensor"
- note removed: "USB-BLE"
- moved on the sheet: C41, D10, D11, D12, D9, R12, R13, R14, R15, R16, R17, R18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

Commit message: PCB: parts placed
Parts:
- removed C6, C7: 22p, Capacitor_SMD:C_0402_1005Metric_Pad0.74x0.62mm_HandSolder, symbol Device:C
- removed Y2: Crystal, Crystal:Crystal_SMD_3215-2Pin_3.2x1.5mm, symbol Device:Crystal
- added C20, C21, C23, C25: 0.1u, Capacitor_SMD:C_0402_1005Metric_Pad0.74x0.62mm_HandSolder, symbol Device:C
- added C22, C26: 4.7u, Capacitor_SMD:C_0603_1608Metric_Pad1.08x0.95mm_HandSolder, symbol Device:C
- added D12, D13: LED, LED_SMD:LED_0603_1608Metric_Pad1.05x0.95mm_HandSolder, symbol Device:LED
- added J10: Conn_01x05_Socket, Connector_PinSocket_2.54mm:PinSocket_1x05_P2.54mm_Vertical, symbol Connector:Conn_01x05_Socket
- added J3: USB_C_Receptacle_USB2.0_16P, Connector_USB:USB_C_Receptacle_HRO_TYPE-C-31-M-12, symbol Connector:USB_C_Receptacle_USB2.0_16P
- added R23, R24: 4.7k, Resistor_SMD:R_0402_1005Metric_Pad0.72x0.64mm_HandSolder, symbol Device:R
- added R25, R26: 470, Resistor_SMD:R_0603_1608Metric_Pad0.98x0.95mm_HandSolder, symbol Device:R
- added U7: FT231XS, Package_SO:SSOP-20_3.9x8.7mm_P0.635mm, symbol Interface_USB:FT231XS
- D5: renamed from D6; value Green -> Red
- J1: footprint Connector_AMASS:AMASS_XT30PW-M_1x02_P2.50mm_Horizontal -> Connector_AMASS:AMASS_XT30U-M_1x02_P5.0mm_Vertical
- R18: renamed from R11; footprint Resistor_SMD:R_0603_1608Metric_Pad0.98x0.95mm_HandSolder -> Resistor_SMD:R_0402_1005Metric_Pad0.72x0.64mm_HandSolder
- R4, R5, R6: footprint Resistor_SMD:R_0603_1608Metric_Pad0.98x0.95mm_HandSolder -> Resistor_SMD:R_0402_1005Metric_Pad0.72x0.64mm_HandSolder
- R7: renamed from R8; footprint Resistor_SMD:R_0603_1608Metric_Pad0.98x0.95mm_HandSolder -> Resistor_SMD:R_0402_1005Metric_Pad0.72x0.64mm_HandSolder
- R8: renamed from R9; footprint Resistor_SMD:R_0603_1608Metric_Pad0.98x0.95mm_HandSolder -> Resistor_SMD:R_0402_1005Metric_Pad0.72x0.64mm_HandSolder
- R9: renamed from R10; footprint Resistor_SMD:R_0603_1608Metric_Pad0.98x0.95mm_HandSolder -> Resistor_SMD:R_0402_1005Metric_Pad0.72x0.64mm_HandSolder
- renumbered C12 to C10, C13 to C11, C41 to C12, C14 to C13, C15 to C14, C16 to C15, C17 to C16, C18 to C17, C19 to C18, C20 to C19, C35 to C27, C37 to C28, C39 to C29, C36 to C30, C38 to C31, C40 to C32, C8 to C6, C9 to C7, C10 to C8, C11 to C9, D11 to D10, D12 to D11, D7 to D6, D8 to D7, D9 to D8, D10 to D9, JP3 to JP2, JP4 to JP3, JP5 to JP4, JP6 to JP5, R12 to R10, R13 to R11, R14 to R12, R15 to R13, R16 to R14, R17 to R15, R18 to R16, R19 to R17, R21 to R19, R22 to R20, R23 to R21, R24 to R22, Y3 to Y2
Connections:
- net I2C3_SDA is gone; now on net BLE_UART_MODE: U3.41 (PC9)
- net +3.3V: now also C23.1, C25.1, C26.1, D12.2 (A), D13.2 (A), U7.13 (3V3OUT), U7.14 (~{RESET}), U7.15 (VCC), U7.3 (VCCIO)
- net BLE_UART_CTS: now also J10.4 (Pin_4)
- net BLE_UART_RTS: now also J10.3 (Pin_3)
- net BLE_UART_RX: now also J10.2 (Pin_2)
- net BLE_UART_TX: now also J10.1 (Pin_1)
- net DIP_1: now also U3.10 (PC2); no longer U3.11 (PC3)
- net DIP_2: now also U3.11 (PC3); no longer U3.12 (PA0)
- net DIP_3: now also U3.12 (PA0); no longer U3.13 (PA1)
- net DIP_4: now also U3.13 (PA1); no longer U3.17 (PA3)
- net GND: now also C20.2, C21.2, C22.2, C23.2, C25.2, C26.2, J10.5 (Pin_5), J3.A1 (GND), J3.A12 (GND), J3.B1 (GND), J3.B12 (GND), R23.2, R24.2, U7.16 (GND), U7.6 (GND)
- net VBUS: now also C20.1, C21.1, C22.1, J3.A4 (VBUS), J3.A9 (VBUS), J3.B4 (VBUS), J3.B9 (VBUS)
- net USART2_TX: now reaches U3.14 (PA2)
- net USART2_TX: now also U7.4 (RXD)
- net I2C3_SCL: no longer names the net of U3.40 (PC8)
- net LPUART1_RX: no longer names the net of U3.8 (PC0)
- net LPUART1_TX: no longer names the net of U3.9 (PC1)
- new net: D13.1 (K), R26.1
- new net: R26.2, U7.10 (CBUS2)
- new net: J3.A6 (D+), J3.B6 (D+), U7.11 (USBDP)
- new net: J3.A7 (D-), J3.B7 (D-), U7.12 (USBDM)
- new net: R25.2, U7.17 (CBUS1)
- new net: J3.A5 (CC1), R23.1
- new net: D12.1 (K), R25.1
- new net: J3.B5 (CC2), R24.1
- new net USART2_RX: U3.17 (PA3), U7.20 (TXD)
- no-connect marks 26 -> 40
Other:
- moved on the sheet: C27, C28, C29, C30, C31, C32, J4, J5, JP2, JP3, JP4, JP5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
