File: KiCad/GN10Mainboard/GN10Mainboard.kicad_pcb (KiCad board)
At the start: 2 copper layers, 70 x 50 mm, 105 parts, among them J1 XT30PW-M, J2 Conn_01x02_Pin, J3 USB_C_Receptacle_USB2.0_16P, J4 Conn_01x04, J5 Conn_01x04, J6 Conn_01x04, J7 Conn_01x04, J8 Conn_01x04, J9 Conn_01x06, SW1 SW_Push, SW2 SW_DIP_x04, SW3 SW_Push, U1 OKL-T/x-W5N-C, U2 3.3V, U3 STM32G474RCTx, U4 TBD62083AFNG, U5 7segmentLED, U6 RNBD451, U7 FT231XS, U8 MCP2562-E-SN, U9 MCP2562-E-SN, Y1 24MHz, Y2 32.768kHz

Commit message: update:schematic
Parts:
- removed G***: LOGO, GN10_Parts:ararobo_6
- removed JP4, JP5: SolderJumper_2_Open, Jumper:SolderJumper-2_P1.3mm_Open_RoundedPad1.0x1.5mm
- removed REF** (x4): MountingHole_3.2mm_M3, MountingHole:MountingHole_3.2mm_M3
- removed TP1, TP2: TestPoint, TestPoint:TestPoint_Pad_D1.0mm
- added C24: 0.1u, Capacitor_SMD:C_0402_1005Metric_Pad0.74x0.62mm_HandSolder, F.Cu at (180.0, 109.2)
- added C33: 18p, Capacitor_SMD:C_0402_1005Metric_Pad0.74x0.62mm_HandSolder, F.Cu at (183.2, 101.3)
- added C34: 0.1u, Capacitor_SMD:C_0402_1005Metric_Pad0.74x0.62mm_HandSolder, F.Cu at (183.2, 103.2)
- added C35: 4.7u, Capacitor_SMD:C_0402_1005Metric_Pad0.74x0.62mm_HandSolder, F.Cu at (183.2, 105.2)
- added C36: 10n, Capacitor_SMD:C_0402_1005Metric_Pad0.74x0.62mm_HandSolder, F.Cu at (183.2, 107.2)
- added C37: 4.7u, Capacitor_SMD:C_0402_1005Metric_Pad0.74x0.62mm_HandSolder, F.Cu at (183.2, 109.2)
- added C38: 6.8n, Capacitor_SMD:C_0402_1005Metric_Pad0.74x0.62mm_HandSolder, F.Cu at (183.2, 111.1)
- added C39: 10n, Capacitor_SMD:C_0402_1005Metric_Pad0.74x0.62mm_HandSolder, F.Cu at (183.2, 113.1)
- added C40: 6.8n, Capacitor_SMD:C_0402_1005Metric_Pad0.74x0.62mm_HandSolder, F.Cu at (183.2, 115.1)
- added C41: 10n, Capacitor_SMD:C_0402_1005Metric_Pad0.74x0.62mm_HandSolder, F.Cu at (186.4, 97.3)
- added C42: 22n, Capacitor_SMD:C_0402_1005Metric_Pad0.74x0.62mm_HandSolder, F.Cu at (186.4, 99.3)
- added C43: 0.1u, Capacitor_SMD:C_0402_1005Metric_Pad0.74x0.62mm_HandSolder, F.Cu at (186.4, 101.3)
- added C44: 10u, Capacitor_SMD:C_0805_2012Metric_Pad1.18x1.45mm_HandSolder, F.Cu at (203.8, 86.9)
- added C45: 10u, Capacitor_SMD:C_0805_2012Metric_Pad1.18x1.45mm_HandSolder, F.Cu at (203.8, 89.9)
- added C46: 0.1u, Capacitor_SMD:C_0402_1005Metric_Pad0.74x0.62mm_HandSolder, F.Cu at (186.4, 103.2)
- added C47: 0.1u, Capacitor_SMD:C_0402_1005Metric_Pad0.74x0.62mm_HandSolder, F.Cu at (186.4, 105.2)
- added C48: 1u, Capacitor_SMD:C_0402_1005Metric_Pad0.74x0.62mm_HandSolder, F.Cu at (186.4, 107.2)
- added C49: 0.1u, Capacitor_SMD:C_0402_1005Metric_Pad0.74x0.62mm_HandSolder, F.Cu at (186.4, 109.2)
- added C50: 1u, Capacitor_SMD:C_0402_1005Metric_Pad0.74x0.62mm_HandSolder, F.Cu at (186.4, 111.1)
- added C51: 0.1u, Capacitor_SMD:C_0402_1005Metric_Pad0.74x0.62mm_HandSolder, F.Cu at (186.4, 113.1)
- added C52: 0.1u, Capacitor_SMD:C_0402_1005Metric_Pad0.74x0.62mm_HandSolder, F.Cu at (186.4, 115.1)
- added C53: 0.1u, Capacitor_SMD:C_0402_1005Metric_Pad0.74x0.62mm_HandSolder, F.Cu at (189.6, 97.3)
- added C54: 0.1u, Capacitor_SMD:C_0402_1005Metric_Pad0.74x0.62mm_HandSolder, F.Cu at (189.6, 99.3)
- added C55: 0.1u, Capacitor_SMD:C_0402_1005Metric_Pad0.74x0.62mm_HandSolder, F.Cu at (189.6, 101.3)
- added C56: 0.1u, Capacitor_SMD:C_0402_1005Metric_Pad0.74x0.62mm_HandSolder, F.Cu at (189.6, 103.2)
- added C57: 0.1u, Capacitor_SMD:C_0402_1005Metric_Pad0.74x0.62mm_HandSolder, F.Cu at (189.6, 105.2)
- added C58: 22p, Capacitor_SMD:C_0402_1005Metric_Pad0.74x0.62mm_HandSolder, F.Cu at (189.6, 107.2)
- added C59: 22p, Capacitor_SMD:C_0402_1005Metric_Pad0.74x0.62mm_HandSolder, F.Cu at (189.6, 109.2)
- added C60: 22p, Capacitor_SMD:C_0402_1005Metric_Pad0.74x0.62mm_HandSolder, F.Cu at (189.6, 111.1)
- added C61: 22p, Capacitor_SMD:C_0402_1005Metric_Pad0.74x0.62mm_HandSolder, F.Cu at (189.6, 113.1)
- added J10: USB_C_Receptacle_USB2.0, Connector_USB:USB_C_Receptacle_HRO_TYPE-C-31-M-12, F.Cu at (181.0, 137.4)
- added J11: Conn_01x06, Connector_JST:JST_XH_B6B-XH-A_1x06_P2.50mm_Vertical, F.Cu at (178.7, 127.2)
- added J12: Conn_01x04, Connector_JST:JST_XH_B4B-XH-A_1x04_P2.50mm_Vertical, F.Cu at (144.1, 109.7)
- added L1: L, Inductor_SMD:L_0603_1608Metric_Pad1.05x0.95mm_HandSolder, F.Cu at (199.3, 71.1)
- added L2: L, Inductor_SMD:L_0603_1608Metric_Pad1.05x0.95mm_HandSolder, F.Cu at (199.3, 73.6)
- added R27: 4.7k, Resistor_SMD:R_0402_1005Metric_Pad0.72x0.64mm_HandSolder, F.Cu at (199.4, 99.3)
- added R28: 4.7k, Resistor_SMD:R_0402_1005Metric_Pad0.72x0.64mm_HandSolder, F.Cu at (199.4, 101.3)
- added R29: 1k, Resistor_SMD:R_0402_1005Metric_Pad0.72x0.64mm_HandSolder, F.Cu at (199.4, 103.3)
- added R30: 12k, Resistor_SMD:R_0402_1005Metric_Pad0.72x0.64mm_HandSolder, F.Cu at (199.4, 105.3)
- added R31: R, Resistor_SMD:R_0402_1005Metric_Pad0.72x0.64mm_HandSolder, F.Cu at (199.4, 107.3)
- added R32: R, Resistor_SMD:R_0402_1005Metric_Pad0.72x0.64mm_HandSolder, F.Cu at (199.4, 109.3)
- added R33: 2.2k, Resistor_SMD:R_0402_1005Metric_Pad0.72x0.64mm_HandSolder, F.Cu at (199.4, 111.3)
- added R34: 2.2k, Resistor_SMD:R_0402_1005Metric_Pad0.72x0.64mm_HandSolder, F.Cu at (199.4, 113.3)
- added R35: 10k, Resistor_SMD:R_0402_1005Metric_Pad0.72x0.64mm_HandSolder, F.Cu at (202.6, 97.3)
- added R36: 10k, Resistor_SMD:R_0402_1005Metric_Pad0.72x0.64mm_HandSolder, F.Cu at (202.6, 99.3)
- added R37: 10k, Resistor_SMD:R_0402_1005Metric_Pad0.72x0.64mm_HandSolder, F.Cu at (202.6, 101.3)
- added R38: 2.2k, Resistor_SMD:R_0402_1005Metric_Pad0.72x0.64mm_HandSolder, F.Cu at (202.6, 103.3)
- added R39: 2.2k, Resistor_SMD:R_0402_1005Metric_Pad0.72x0.64mm_HandSolder, F.Cu at (202.6, 105.3)
- added U10: BNO086, Package_LGA:LGA-28_5.2x3.8mm_P0.5mm, F.Cu at (213.5, 126.2)
- added Y3: 25M, Crystal:Crystal_SMD_2016-4Pin_2.0x1.6mm, F.Cu at (142.5, 141.7)
- added Y4: 12M, Crystal:Resonator_SMD_Murata_CSTxExxV-3Pin_3.0x1.1mm_HandSoldering, F.Cu at (208.8, 74.4)
- added Y6: 32.768kHz, Crystal:Crystal_SMD_3215-2Pin_3.2x1.5mm, F.Cu at (189.4, 136.7)
- added Y7: 32.768kHz, Crystal:Crystal_SMD_3215-2Pin_3.2x1.5mm, F.Cu at (189.4, 140.0)
- C12, C18: value 0.1u -> 10u; footprint Capacitor_SMD:C_0402_1005Metric_Pad0.74x0.62mm_HandSolder -> Capacitor_SMD:C_0805_2012Metric_Pad1.18x1.45mm_HandSolder
- C13, C19: value 10u -> 0.1u; footprint Capacitor_SMD:C_0805_2012Metric_Pad1.18x1.45mm_HandSolder -> Capacitor_SMD:C_0402_1005Metric_Pad0.74x0.62mm_HandSolder
- C16: value 0.1u -> 18p
- C17: value 18p -> 0.1u
- C22: value 4.7u -> 0.1u; footprint Capacitor_SMD:C_0603_1608Metric_Pad1.08x0.95mm_HandSolder -> Capacitor_SMD:C_0402_1005Metric_Pad0.74x0.62mm_HandSolder
- C25, C27: value 0.1u -> 100u; footprint Capacitor_SMD:C_0402_1005Metric_Pad0.74x0.62mm_HandSolder -> Capacitor_THT:CP_Radial_D6.3mm_P2.50mm
- C26: value 4.7u -> 100u; footprint Capacitor_SMD:C_0603_1608Metric_Pad1.08x0.95mm_HandSolder -> Capacitor_THT:CP_Radial_D6.3mm_P2.50mm
- C28: value 0.1u -> 1u
- C29: value 100u -> 0.1u; footprint Capacitor_THT:CP_Radial_D6.3mm_P2.50mm -> Capacitor_SMD:C_0402_1005Metric_Pad0.74x0.62mm_HandSolder
- C32: value 100u -> 18p; footprint Capacitor_THT:CP_Radial_D6.3mm_P2.50mm -> Capacitor_SMD:C_0402_1005Metric_Pad0.74x0.62mm_HandSolder
- J3: value USB_C_Receptacle_USB2.0_16P -> Conn_01x04; footprint Connector_USB:USB_C_Receptacle_HRO_TYPE-C-31-M-12 -> Connector_JST:JST_XH_B4B-XH-A_1x04_P2.50mm_Vertical
- J5: value Conn_01x04 -> Conn_01x06; footprint Connector_JST:JST_XH_B4B-XH-A_1x04_P2.50mm_Vertical -> Connector_JST:JST_XH_B6B-XH-A_1x06_P2.50mm_Vertical
- J9: value Conn_01x06 -> RJ45_Bel_SI-60062-F; footprint Connector_JST:JST_XH_B6B-XH-A_1x06_P2.50mm_Vertical -> Connector_RJ:RJ45_Bel_SI-60062-F
- JP2, JP3: value SolderJumper_2_Open -> SolderJumper_3_Open; footprint Jumper:SolderJumper-2_P1.3mm_Open_RoundedPad1.0x1.5mm -> Jumper:SolderJumper-3_P1.3mm_Open_RoundedPad1.0x1.5mm
- R10: value 330 -> 1k; footprint Resistor_SMD:R_0603_1608Metric_Pad0.98x0.95mm_HandSolder -> Resistor_SMD:R_0402_1005Metric_Pad0.72x0.64mm_HandSolder
- R11, R12, R13, R14: value 330 -> 1k
- R15, R16, R17: value 330 -> PU; footprint Resistor_SMD:R_0603_1608Metric_Pad0.98x0.95mm_HandSolder -> Resistor_SMD:R_0402_1005Metric_Pad0.72x0.64mm_HandSolder
- R18: value 1k -> PU
- R19: value 1k -> PU; footprint Resistor_SMD:R_0603_1608Metric_Pad0.98x0.95mm_HandSolder -> Resistor_SMD:R_0402_1005Metric_Pad0.72x0.64mm_HandSolder
- R20, R21, R22: value 1k -> 49; footprint Resistor_SMD:R_0603_1608Metric_Pad0.98x0.95mm_HandSolder -> Resistor_SMD:R_0402_1005Metric_Pad0.72x0.64mm_HandSolder
- R23: value 4.7k -> 12.4k
- R24: value 4.7k -> 49
- R25, R26: value 470 -> R; footprint Resistor_SMD:R_0603_1608Metric_Pad0.98x0.95mm_HandSolder -> Resistor_SMD:R_0402_1005Metric_Pad0.72x0.64mm_HandSolder
- U4: value TBD62083AFNG -> RNBD451; footprint Package_SO:SSOP-18_4.4x6.5mm_P0.65mm -> GN10_Parts:ZSX
- U5: value 7segmentLED -> MCP2562-E-SN; footprint GN10_Parts:OSL10326 -> Package_SO:SOIC-8_3.9x4.9mm_P1.27mm
- U6: value RNBD451 -> MCP2562-E-SN; footprint GN10_Parts:ZSX -> Package_SO:SOIC-8_3.9x4.9mm_P1.27mm
- U7: value FT231XS -> MCP2562-E-SN; footprint Package_SO:SSOP-20_3.9x8.7mm_P0.635mm -> Package_SO:SOIC-8_3.9x4.9mm_P1.27mm
- U8: value MCP2562-E-SN -> W5500; footprint Package_SO:SOIC-8_3.9x4.9mm_P1.27mm -> Package_QFP:LQFP-48_7x7mm_P0.5mm
- U9: value MCP2562-E-SN -> FT2232HQ; footprint Package_SO:SOIC-8_3.9x4.9mm_P1.27mm -> Package_DFN_QFN:QFN-64-1EP_9x9mm_P0.5mm_EP4.35x4.35mm
- moved SW2 84.1 mm to (211.6, 89.1)
- moved J2 83.1 mm to (212.2, 118.4), turned to 0 degrees
- moved C1 82.3 mm to (203.8, 68.8), turned to 0 degrees
- moved C3 82.3 mm to (203.8, 74.8), turned to 0 degrees
- moved D12 81.9 mm to (215.2, 102.8), turned to 0 degrees
- moved D3 79.3 mm to (206.5, 100.2), turned to 0 degrees
- moved Y1 77.9 mm to (208.8, 69.7), turned to 0 degrees
- moved D13 77.7 mm to (215.2, 105.4), turned to 0 degrees
- moved U2 77.4 mm to (211.2, 81.0)
- moved C11 76.6 mm to (199.3, 68.6), turned to 0 degrees
- moved C12 75.4 mm to (203.8, 80.8), turned to 0 degrees
- moved R11 75.3 mm to (199.3, 83.6), turned to 0 degrees
- moved R12 74.5 mm to (199.3, 86.1), turned to 0 degrees
- moved J1 74.2 mm to (207.9, 110.3), turned to 0 degrees
- moved R1 70.6 mm to (199.3, 76.1)
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Connections:
- C14 pad 1: +3.3V -> BLE_RESET
- C15 pad 1: Net-(U6-PA11) -> Net-(U4-PA11)
- C16 pad 1: BLE_RESET -> Net-(U4-PA12)
- C17 pad 1: Net-(U6-PA12) -> +3.3V
- C20 pad 1: VBUS -> +3.3V
- C21 pad 1: VBUS -> +3.3V
- C22 pad 1: VBUS -> +5V
- C23 pad 1: +3.3V -> +5V
- C25 pad 1: +3.3V -> +5V
- C26 pad 1: +3.3V -> +5V
- C27 pad 1: +3.3V -> +5V
- C28 pad 1: +5V -> +3.3V
- C29 pad 1: +5V -> +3.3V
- C31 pad 1: +5V -> +3.3V
- C32 pad 1: +5V -> Net-(U8-XI/CLKIN)
- J4 pad 1: GND -> +3.3V
- J4 pad 2: CAN1_L -> SYS_SWCLK
- J4 pad 3: +5V -> GND
- J4 pad 4: CAN1_H -> SYS_SWDIO
- J5 pad 1: GND -> TIM1_CH1
- J5 pad 2: CAN2_L -> +3.3V
- J5 pad 3: +5V -> TIM1_CH2
- J5 pad 4: CAN2_H -> GND
- J6 pad 1: USART3_RX -> GND
- J6 pad 2: +3.3V -> CAN1_L
- J6 pad 3: USART3_TX -> +5V
- J6 pad 4: GND -> CAN1_H
- J7 pad 1: I2C4_SCL -> GND
- J7 pad 2: +3.3V -> CAN2_L
- J7 pad 3: I2C4_SDA -> +5V
- J7 pad 4: GND -> CAN2_H
- J8 pad 1: +3.3V -> GND
- J8 pad 2: SYS_SWCLK -> CAN3_L
- J8 pad 3: GND -> +5V
- J8 pad 4: SYS_SWDIO -> CAN3_H
- J9 pad 1: SPI3_MOSI -> Net-(J9-TD+)
- J9 pad 2: +3.3V -> Net-(J9-TCT)
- J9 pad 3: SPI3_MISO -> Net-(J9-TD-)
- J9 pad 4: GND -> Net-(J9-RD+)
- J9 pad 5: SPI3_SCK -> Net-(J9-RCT)
- J9 pad 6: SPI3_CS -> Net-(J9-RD-)
- JP2 pad 1: USART1_RTS -> USART1_RX
- JP2 pad 2: BLE_UART_CTS -> BLE_UART_TX
- JP3 pad 1: BLE_UART_RTS -> USART1_TX
- JP3 pad 2: USART1_CTS -> BLE_UART_RX
- R10 pad 1: Net-(U4-O1) -> Net-(D7-K)
- R10 pad 2: LED_A_DRV -> GND
- R11 pad 1: Net-(U4-O2) -> Net-(D8-K)
- R11 pad 2: LED_B_DRV -> BLE_STATUS_LED
- R12 pad 1: Net-(U4-O3) -> Net-(D9-K)
- R12 pad 2: LED_C_DRV -> BLE_EVENT_LED
- R13 pad 1: Net-(U4-O4) -> Net-(D10-K)
- R13 pad 2: LED_D_DRV -> BLE_UART_TX_LED
- R14 pad 1: Net-(U4-O5) -> Net-(D11-K)
- R14 pad 2: LED_E_DRV -> BLE_UART_RX_LED
- R15 pad 1: Net-(U4-O6) -> +3.3V
- R15 pad 2: LED_F_DRV -> Net-(U8-PMODE0)
- R16 pad 1: Net-(U4-O7) -> +3.3V
- R16 pad 2: LED_G_DRV -> Net-(U8-PMODE1)
- R17 pad 1: Net-(U4-O8) -> +3.3V
- R17 pad 2: LED_DP_DRV -> Net-(U8-PMODE2)
- R18 pad 1: Net-(D7-K) -> +3.3V
- R18 pad 2: GND -> W5500_RST
- R19 pad 1: Net-(D8-K) -> +3.3V
- R19 pad 2: BLE_STATUS_LED -> Net-(U8-~{INT})
- R20 pad 1: Net-(D9-K) -> Net-(U8-RXN)
- R20 pad 2: BLE_EVENT_LED -> Net-(C39-Pad1)
- R21 pad 1: Net-(D10-K) -> +3.3V
- R21 pad 2: BLE_UART_TX_LED -> Net-(J9-TD-)
- R22 pad 1: Net-(D11-K) -> Net-(U8-RXP)
- R22 pad 2: BLE_UART_RX_LED -> Net-(C39-Pad1)
- R23 pad 1: Net-(J3-CC1) -> Net-(U8-EXRES1)
- R24 pad 1: Net-(J3-CC2) -> +3.3V
- R24 pad 2: GND -> Net-(J9-TD+)
- R25 pad 1: Net-(D12-K) -> GND
- R25 pad 2: Net-(U7-CBUS1) -> Net-(J9-PadL1)
- R26 pad 1: Net-(D13-K) -> GND
- R26 pad 2: Net-(U7-CBUS2) -> Net-(J9-PadL3)
- U3 pad 18: LED_DP -> W5500_RST
- U3 pad 19: LED_G -> SPI1_SCK
- U3 pad 20: LED_F -> SPI1_MISO
- U3 pad 21: LED_E -> SPI1_MOSI
- U3 pad 22: LED_D -> SPI1_CS
- U3 pad 23: LED_C -> unconnected-(U3-PC5-Pad23)
- U3 pad 24: LED_B -> BLE_UART_MODE
- U3 pad 25: LED_A -> unconnected-(U3-PB1-Pad25)
- U3 pad 3: unconnected-(U3-PC14-Pad3) -> Net-(U3-PC14)
- U3 pad 38: I2C4_SCL -> TIM3_CH1
- U3 pad 39: I2C4_SDA -> TIM3_CH2
- U3 pad 4: unconnected-(U3-PC15-Pad4) -> Net-(U3-PC15)
- U3 pad 40: unconnected-(U3-PC8-Pad40) -> I2C3_SCL
- U3 pad 41: BLE_UART_MODE -> I2C3_SDA
- U3 pad 45: USART1_CTS -> FDCAN1_RX
- U3 pad 46: USART1_RTS -> FDCAN1_TX
- U3 pad 51: SPI3_CS -> unconnected-(U3-PA15-Pad51)
- U3 pad 52: SPI3_SCK -> SW1
- U3 pad 53: SPI3_MISO -> SW2
- U3 pad 54: SPI3_MOSI -> SW3
- U3 pad 8: unconnected-(U3-PC0-Pad8) -> TIM1_CH1
- U3 pad 9: unconnected-(U3-PC1-Pad9) -> TIM1_CH2
- U4 pad 1: LED_A -> GND
- U4 pad 10: +3.3V -> Net-(U4-PA12)
- U4 pad 11: Net-(U4-O8) -> GND
- U4 pad 12: Net-(U4-O7) -> BLE_UART_RX
- U4 pad 13: Net-(U4-O6) -> unconnected-(U4-PB7-Pad13)
- U4 pad 14: Net-(U4-O5) -> unconnected-(U4-PB8-Pad14)
- U4 pad 15: Net-(U4-O4) -> unconnected-(U4-PB9-Pad15)
- U4 pad 16: Net-(U4-O3) -> unconnected-(U4-PA4-Pad16)
- U4 pad 17: Net-(U4-O2) -> unconnected-(U4-PB10-Pad17)
- U4 pad 18: Net-(U4-O1) -> unconnected-(U4-PB11-Pad18)
- U4 pad 2: LED_B -> GND
- U4 pad 3: LED_C -> BLE_RESET
- U4 pad 4: LED_D -> unconnected-(U4-PB0-Pad4)
- U4 pad 5: LED_E -> unconnected-(U4-PB3-Pad5)
- U4 pad 6: LED_F -> BLE_STATUS_LED
- U4 pad 7: LED_G -> +3.3V
- U4 pad 8: LED_DP -> GND
- U4 pad 9: GND -> Net-(U4-PA11)
- U5 pad 1: LED_A_DRV -> CAN1_TX
- U5 pad 2: LED_F_DRV -> GND
- U5 pad 3: LED_G_DRV -> +5V
- U5 pad 4: LED_E_DRV -> CAN1_RX
- U5 pad 5: LED_D_DRV -> +3.3V
- U5 pad 6: LED_DP_DRV -> CAN1_L
- U5 pad 7: +3.3V -> CAN1_H
- U5 pad 8: LED_C_DRV -> GND
- U6 pad 1: GND -> CAN2_TX
- U6 pad 3: BLE_RESET -> +5V
- U6 pad 4: unconnected-(U6-PB0-Pad4) -> CAN2_RX
- U6 pad 5: unconnected-(U6-PB3-Pad5) -> +3.3V
- U6 pad 6: BLE_STATUS_LED -> CAN2_L
- U6 pad 7: +3.3V -> CAN2_H
- U7 pad 1: unconnected-(U7-~{DTR}-Pad1) -> CAN3_TX
- U7 pad 2: unconnected-(U7-~{RTS}-Pad2) -> GND
- U7 pad 3: +3.3V -> +5V
- U7 pad 4: USART2_TX -> CAN3_RX
- U7 pad 5: unconnected-(U7-~{RI}-Pad5) -> +3.3V
- U7 pad 6: GND -> CAN3_L
- U7 pad 7: unconnected-(U7-~{DSR}-Pad7) -> CAN3_H
- U7 pad 8: unconnected-(U7-~{DCD}-Pad8) -> GND
- U8 pad 1: CAN2_TX -> Net-(J9-TD-)
- U8 pad 2: GND -> Net-(J9-TD+)
- U8 pad 3: +5V -> GND
- U8 pad 4: CAN2_RX -> +3.3V
- U8 pad 5: +3.3V -> Net-(U8-RXN)
- U8 pad 6: CAN1_L -> Net-(U8-RXP)
- U8 pad 7: CAN1_H -> unconnected-(U8-DNC-Pad7)
- U8 pad 8: GND -> +3.3V
- U9 pad 1: CAN3_TX -> GND
- U9 pad 2: GND -> Net-(U9-OSCI)
- U9 pad 3: +5V -> Net-(U9-OSCO)
- U9 pad 4: CAN3_RX -> Net-(U9-VPHY)
- U9 pad 5: +3.3V -> GND
- U9 pad 6: CAN2_L -> Net-(U9-REF)
- U9 pad 7: CAN2_H -> USBD-
- U9 pad 8: GND -> USBD+
- Y2 pad 1: Net-(U6-PA11) -> Net-(U4-PA11)
- Y2 pad 2: Net-(U6-PA12) -> Net-(U4-PA12)
Routing:
- net +3.3V: track 286.5 -> 0.00 mm, vias 12 -> 0
- net +5V: track 146.6 -> 0.00 mm, vias 2 -> 0
- net SPI3_MOSI: track 37.7 -> 0.00 mm, vias 1 -> 0
- net SPI3_MISO: track 33.1 -> 0.00 mm, vias 1 -> 0
- net DIP_1: track 29.6 -> 0.00 mm, vias 2 -> 0
- net SYS_SWCLK: track 29.6 -> 0.00 mm, vias 1 -> 0
- net DIP_2: track 29.2 -> 0.00 mm, vias 2 -> 0
- net DIP_3: track 28.7 -> 0.00 mm, vias 2 -> 0
- net SPI3_SCK: track 28.5 -> 0.00 mm, vias 1 -> 0
- net DIP_4: track 28.3 -> 0.00 mm, vias 2 -> 0
- net BLE_RESET: track 27.4 -> 0.00 mm
- net SYS_SWDIO: track 26.8 -> 0.00 mm, vias 1 -> 0
- net SPI3_CS: track 26.4 -> 0.00 mm, vias 1 -> 0
- net BLE_UART_MODE: track 26.0 -> 0.00 mm, vias 2 -> 0
- net GND: track 25.3 -> 0.00 mm, vias 287 -> 0
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- removed copper zone on F.Cu, net +3.3V
- removed copper zone on F.Cu, net +5V
- removed copper zone on F.Cu, net +BATT
- removed copper zone on B.Cu, net GND
- removed copper zone on F.Cu, net GND
Other:
- board outline removed
- board text removed: "5V"
- board text removed: "5V-VBUS"
- board text removed: "BLE"
- board text removed: "BLE_RST"
- board text removed: "CAN2"
- board text removed: "CAN3"
- board text removed: "CTS"
- board text removed: "GN10Mainboard v1.1"
- board text removed: "I2C"
- board text removed: "RST"
- board text removed: "RTS"
- board text removed: "RX"
- board text removed: "RX TX"
- board text removed: "SPI"
- board text removed: "STATUS"
- board text removed: "STLink"
- board text removed: "STM32"
- board text removed: "TX"
- board text removed: "TX RX EVENT"
- board text removed: "UART"
- board text removed: "https://github.com/ararobo/GN10Mainboard designed by: GN10/Gento Aiba"

Commit message: update:PCB
Parts:
- removed C25, C26, C27: 100u, Capacitor_THT:CP_Radial_D6.3mm_P2.50mm
- removed D10: Blue, LED_SMD:LED_0603_1608Metric_Pad1.05x0.95mm_HandSolder
- removed D11: Green, LED_SMD:LED_0603_1608Metric_Pad1.05x0.95mm_HandSolder
- removed JP1: SolderJumper_2_Open, Jumper:SolderJumper-2_P1.3mm_Open_RoundedPad1.0x1.5mm
- removed R1: 20k, Resistor_SMD:R_0603_1608Metric_Pad0.98x0.95mm_HandSolder
- removed R13, R14: 1k, Resistor_SMD:R_0603_1608Metric_Pad0.98x0.95mm_HandSolder
- added REF**: MountingHole_3.2mm_M3, MountingHole:MountingHole_3.2mm_M3, F.Cu at (133.6, 93.6)
- added REF**: MountingHole_3.2mm_M3, MountingHole:MountingHole_3.2mm_M3, F.Cu at (206.4, 146.4)
- added REF**: MountingHole_3.2mm_M3, MountingHole:MountingHole_3.2mm_M3, F.Cu at (206.4, 93.6)
- added REF**: MountingHole_3.2mm_M3, MountingHole:MountingHole_3.2mm_M3, F.Cu at (133.6, 146.4)
- C44, C45: footprint Capacitor_SMD:C_0805_2012Metric_Pad1.18x1.45mm_HandSolder -> Resistor_SMD:R_0603_1608Metric_Pad0.98x0.95mm_HandSolder
- JP2, JP3: moved to B.Cu
- moved J3 83.4 mm to (178.1, 146.8), turned to 180 degrees
- moved SW2 82.1 mm to (135.5, 119.8)
- moved SW3 79.6 mm to (134.2, 114.2)
- moved C1 74.1 mm to (194.0, 142.3), turned to 180 degrees
- moved Y4 73.1 mm to (146.5, 112.6), turned to -90 degrees
- moved L1 72.9 mm to (145.5, 120.3)
- moved D8 72.3 mm to (139.3, 92.5), turned to -90 degrees
- moved C2 72.2 mm to (187.9, 142.3)
- moved J2 71.8 mm to (140.7, 111.3), turned to 180 degrees
- moved L2 69.3 mm to (145.5, 117.2)
- moved Y1 67.7 mm to (166.7, 122.7), turned to -90 degrees
- moved JP2 66.6 mm to (161.3, 109.9)
- moved J4 66.5 mm to (206.7, 100.8), turned to -90 degrees
- moved C44 66.5 mm to (145.5, 118.8), turned to 180 degrees
- moved U2 66.3 mm to (178.9, 139.0), turned to 180 degrees
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Connections:
- J10 pad A4: +5V -> VBUS
- J10 pad A9: +5V -> VBUS
- J10 pad B4: +5V -> VBUS
- J10 pad B9: +5V -> VBUS
- U1 pad 1: Net-(JP1-B) -> GND
- U3 pad 45: FDCAN1_RX -> CAN1_RX
- U3 pad 46: FDCAN1_TX -> CAN1_TX
Routing:
- net +3.3V: track 0.00 -> 168.7 mm
- net +5V: track 0.00 -> 60.2 mm, vias 0 -> 1
- net DIP_1: track 0.00 -> 48.7 mm, vias 0 -> 2
- net DIP_2: track 0.00 -> 48.3 mm, vias 0 -> 2
- net DIP_3: track 0.00 -> 47.9 mm, vias 0 -> 2
- net DIP_4: track 0.00 -> 47.5 mm, vias 0 -> 2
- net STM32_RESET: track 0.00 -> 47.1 mm, vias 0 -> 2
- net TIM1_CH1: track 0.00 -> 44.8 mm, vias 0 -> 1
- net TIM1_CH2: track 0.00 -> 41.0 mm, vias 0 -> 1
- net TIM3_CH1: track 0.00 -> 37.5 mm, vias 0 -> 1
- net USART2_RX: track 0.00 -> 35.5 mm, vias 0 -> 2
- net TIM3_CH2: track 0.00 -> 34.7 mm, vias 0 -> 1
- net BLE_RESET: track 0.00 -> 34.4 mm
- net SYS_SWCLK: track 0.00 -> 33.8 mm
- net CAN3_TX: track 0.00 -> 33.1 mm
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- added copper zone on B.Cu, net GND
- added copper zone on F.Cu, net GND
- added copper zone on In1.Cu, net GND
Other:
- board outline added: 80 x 66 mm
- copper layers 2 -> 4

Commit message: update:PCB
Parts:
- added G***: LOGO, GN10_Parts:ararobosmall, F.Cu at (190.8, 109.6)
- moved R8 24.4 mm to (183.3, 131.8), turned to -90 degrees
- moved C24 23.9 mm to (182.1, 112.7), turned to 180 degrees
- moved R9 22.5 mm to (184.5, 131.8), turned to -90 degrees
- moved J6 22.0 mm to (169.3, 93.9), turned to -90 degrees
- moved R10 21.4 mm to (185.6, 131.8), turned to -90 degrees
- moved D5 20.9 mm to (183.0, 128.9), turned to 90 degrees
- moved D6 19.7 mm to (184.5, 128.9), turned to 90 degrees
- moved U7 17.8 mm to (182.1, 108.3), turned to 90 degrees
- moved D7 17.7 mm to (186.0, 128.9), turned to 90 degrees
- moved J4 16.3 mm to (192.0, 93.9)
- moved C21 15.7 mm to (185.4, 106.4), turned to -90 degrees
- moved C23 14.3 mm to (175.1, 112.7), turned to 180 degrees
- moved J7 12.3 mm to (176.4, 93.9), turned to -90 degrees
- moved J11 8.79 mm to (207.0, 100.4)
- moved J5 8.78 mm to (200.1, 100.4)
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Routing:
- net +3.3V: track 168.7 -> 457.4 mm, vias 0 -> 14
- net +5V: track 60.2 -> 138.2 mm
- net SW3: track 0.00 -> 60.1 mm, vias 0 -> 1
- net SW2: track 0.00 -> 57.7 mm, vias 0 -> 1
- net SW1: track 0.00 -> 55.3 mm, vias 0 -> 1
- net BLE_UART_MODE: track 0.00 -> 51.1 mm, vias 0 -> 2
- net ACT: track 0.00 -> 40.6 mm, vias 0 -> 1
- net LNK: track 0.00 -> 36.2 mm, vias 0 -> 1
- net +1V8: track 6.08 -> 32.2 mm
- net USBD+: track 0.00 -> 25.5 mm, vias 0 -> 2
- net USBD-: track 0.00 -> 24.1 mm, vias 0 -> 2
- net CAN3_TX: track 33.1 -> 8.95 mm
- net LED_RED: track 26.7 -> 2.66 mm, vias 2 -> 0
- net GNDS: track 0.00 -> 22.6 mm
- net LED_GREEN: track 26.2 -> 4.53 mm, vias 2 -> 0
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- added copper zone on F.Cu, net +5V
- added copper zone on F.Cu, net +BATT
Other:
- outline, holes or cut-outs redrawn
- board text added: "3 2 1"
- board text added: "5V"
- board text added: "BATT"
- board text added: "BLE"
- board text added: "CAN1"
- board text added: "CAN2"
- board text added: "CAN3"
- board text added: "EVENT"
- board text added: "MCU"
- board text added: "STATUS"
- board text added: "STLink"
- board text added: "Switch"
- board text added: "UART"
- board text added: "VBUS"
